File: Right/Tastatur.kicad_pcb (KiCad board)
At the start: 2 copper layers, 663.8 x 129.9 mm, 145 parts, among them J101 Conn_01x04_Pin, J102 XT60PW-F, Q101 SI2301CDS-T1-GE3, Q102 SI2301CDS-T1-GE3, Q103 SI2301CDS-T1-GE3, Q104 SI2301CDS-T1-GE3, Q105 SI2301CDS-T1-GE3, Q106 2N7002HW, Q107 SI2301CDS-T1-GE3, SW101 MK-12C02-G020, SW201 SW_Push, SW202 SW_Push, SW203 SW_Push, SW204 SW_Push, SW205 SW_Push, SW206 SW_Push, SW207 SW_Push, SW208 SW_Push, SW209 SW_Push, SW210 SW_Push, SW211 SW_Push, SW212 SW_Push, SW213 SW_Push, SW214 SW_Push, SW215 SW_Push, SW216 SW_Push, SW217 SW_Push, SW218 SW_Push, SW219 SW_Push, U101 USBLC6-2SC6, U102 CH592F, U103 AP2112K-3.3, U104 MT3608, U105 TP4056-42-ESOP8, U106 CD4052B, U107 LM393, Y101 32MHz

Commit message: redesign with smaller components
Parts:
- removed AE101: Antenna_Shield, Inductor_SMD:L_1206_3216Metric
- removed C101: 470n, Capacitor_SMD:C_0603_1608Metric_Pad1.08x0.95mm_HandSolder
- removed C102: 4u7, Capacitor_SMD:C_0603_1608Metric_Pad1.08x0.95mm_HandSolder
- removed C103: 100n, Capacitor_SMD:C_0603_1608Metric_Pad1.08x0.95mm_HandSolder
- removed C104: 2u2, Capacitor_SMD:C_0603_1608Metric_Pad1.08x0.95mm_HandSolder
- removed C105, C106: 10p, Capacitor_SMD:C_0603_1608Metric_Pad1.08x0.95mm_HandSolder
- removed C111: 10u, Capacitor_SMD:C_0603_1608Metric_Pad1.08x0.95mm_HandSolder
- removed D103: GREEN, LED_SMD:LED_0603_1608Metric
- removed D104: RED, LED_SMD:LED_0603_1608Metric
- removed DL201, DL202, DL203, DL204, DL205, DL206, DL207, DL208, DL209, DL210, DL211, DL212, DL213, DL214, DL215, DL216, DL217, DL218, DL219: SK6805-EC15, LED_SMD:LED_SK6812_EC15_1.5x1.5mm
- removed H101, H102: MountingHole, MountingHole:MountingHole_2.2mm_M2_ISO7380
- removed J101: Conn_01x04_Pin, Connector_JST:JST_PH_B4B-PH-K_1x04_P2.00mm_Vertical
- removed J102: XT60PW-F, Connector_AMASS:AMASS_XT60PW-F_1x02_P7.20mm_Horizontal
- removed L101: 10u, Inductor_SMD:L_0603_1608Metric_Pad1.05x0.95mm_HandSolder
- removed Q101, Q102, Q103, Q104, Q105, Q107: SI2301CDS-T1-GE3, Package_TO_SOT_SMD:SOT-23_Handsoldering
- removed Q106: 2N7002HW, Package_TO_SOT_SMD:SOT-323_SC-70_Handsoldering
- removed R106: 15k, Resistor_SMD:R_0603_1608Metric_Pad0.98x0.95mm_HandSolder
- removed R107, R115: 330R, Resistor_SMD:R_0603_1608Metric_Pad0.98x0.95mm_HandSolder
- removed R109: 50k, Resistor_SMD:R_0603_1608Metric_Pad0.98x0.95mm_HandSolder
- removed SW101: MK-12C02-G020, Button_Switch_SMD:SW_SPDT_PCM12
- removed TP102: TestPoint, TestPoint:TestPoint_Pad_D1.0mm
- removed U102: CH592F, steew:CH592F
- removed U105: TP4056-42-ESOP8, Package_SO:SOP-8-1EP_4.57x4.57mm_P1.27mm_EP4.57x4.45mm
- removed U106: CD4052B, Package_SO:TSSOP-16_4.4x5mm_P0.65mm
- removed Y101: 32MHz, Crystal:Crystal_SMD_2016-4Pin_2.0x1.6mm
- added AE1: Antenna_Shield, Inductor_SMD:L_1206_3216Metric, F.Cu at (187.0, 110.8)
- added C1: 4u7, Capacitor_SMD:C_0402_1005Metric_Pad0.74x0.62mm_HandSolder, F.Cu at (174.8, 106.4)
- added C2: 1u, Capacitor_SMD:C_0402_1005Metric_Pad0.74x0.62mm_HandSolder, F.Cu at (183.0, 100.5)
- added C3: 100p, Capacitor_SMD:C_0402_1005Metric_Pad0.74x0.62mm_HandSolder, F.Cu at (184.0, 100.5)
- added C35: 1p, Capacitor_SMD:C_0402_1005Metric_Pad0.74x0.62mm_HandSolder, F.Cu at (185.2, 106.5)
- added C36: 802p, Capacitor_SMD:C_0402_1005Metric_Pad0.74x0.62mm_HandSolder, F.Cu at (180.8, 110.5)
- added C37: 4u7, Capacitor_SMD:C_0402_1005Metric_Pad0.74x0.62mm_HandSolder, F.Cu at (175.8, 110.5)
- added C38: 4u7, Capacitor_SMD:C_0402_1005Metric_Pad0.74x0.62mm_HandSolder, F.Cu at (173.8, 110.5)
- added C39: 4u7, Capacitor_SMD:C_0402_1005Metric_Pad0.74x0.62mm_HandSolder, F.Cu at (174.8, 110.5)
- added C4: 100n, Capacitor_SMD:C_0402_1005Metric_Pad0.74x0.62mm_HandSolder, F.Cu at (176.8, 110.5)
- added C40: 1p2, Capacitor_SMD:C_0402_1005Metric_Pad0.74x0.62mm_HandSolder, F.Cu at (186.2, 106.5)
- added C41: 12p, Capacitor_SMD:C_0402_1005Metric_Pad0.74x0.62mm_HandSolder, F.Cu at (175.2, 102.4)
- added C42: 12p, Capacitor_SMD:C_0402_1005Metric_Pad0.74x0.62mm_HandSolder, F.Cu at (175.2, 104.7)
- added C43: 10u, Capacitor_SMD:C_0402_1005Metric_Pad0.74x0.62mm_HandSolder, F.Cu at (192.2, 126.8)
- added C5: 100n, Capacitor_SMD:C_0402_1005Metric_Pad0.74x0.62mm_HandSolder, F.Cu at (173.5, 101.2)
- added C6: 10p, Capacitor_SMD:C_0402_1005Metric_Pad0.74x0.62mm_HandSolder, F.Cu at (186.0, 103.5)
- added C9: 10p, Capacitor_SMD:C_0402_1005Metric_Pad0.74x0.62mm_HandSolder, F.Cu at (186.8, 99.8)
- added D10: SK6805-EC15, LED_SMD:LED_SK6812_EC15_1.5x1.5mm, F.Cu at (143.1, 72.6)
- added D11: SK6805-EC15, LED_SMD:LED_SK6812_EC15_1.5x1.5mm, F.Cu at (163.1, 75.1)
- added D17: SK6805-EC15, LED_SMD:LED_SK6812_EC15_1.5x1.5mm, F.Cu at (83.1, 95.1)
- added D18: SK6805-EC15, LED_SMD:LED_SK6812_EC15_1.5x1.5mm, F.Cu at (103.1, 92.6)
- added D19: SK6805-EC15, LED_SMD:LED_SK6812_EC15_1.5x1.5mm, F.Cu at (123.1, 90.1)
- added D20: SK6805-EC15, LED_SMD:LED_SK6812_EC15_1.5x1.5mm, F.Cu at (143.1, 92.6)
- added D21: SK6805-EC15, LED_SMD:LED_SK6812_EC15_1.5x1.5mm, F.Cu at (163.1, 95.1)
- added D27: SK6805-EC15, LED_SMD:LED_SK6812_EC15_1.5x1.5mm, F.Cu at (83.1, 115.1)
- added D28: SK6805-EC15, LED_SMD:LED_SK6812_EC15_1.5x1.5mm, F.Cu at (103.1, 112.6)
- added D29: SK6805-EC15, LED_SMD:LED_SK6812_EC15_1.5x1.5mm, F.Cu at (123.1, 110.1)
- added D30: SK6805-EC15, LED_SMD:LED_SK6812_EC15_1.5x1.5mm, F.Cu at (143.1, 112.6)
- added D31: SK6805-EC15, LED_SMD:LED_SK6812_EC15_1.5x1.5mm, F.Cu at (163.1, 115.1)
- added D37: SK6805-EC15, LED_SMD:LED_SK6812_EC15_1.5x1.5mm, F.Cu at (103.1, 132.6)
- added D38: SK6805-EC15, LED_SMD:LED_SK6812_EC15_1.5x1.5mm, F.Cu at (123.1, 130.1)
- added D39: SK6805-EC15, LED_SMD:LED_SK6812_EC15_1.5x1.5mm, F.Cu at (143.1, 132.6)
- added D40: SK6805-EC15, LED_SMD:LED_SK6812_EC15_1.5x1.5mm, F.Cu at (163.1, 135.1)
- added D45: GREEN, LED_SMD:LED_0603_1608Metric, F.Cu at (192.6, 124.5)
- added D7: SK6805-EC15, LED_SMD:LED_SK6812_EC15_1.5x1.5mm, F.Cu at (83.1, 75.1)
- added D8: SK6805-EC15, LED_SMD:LED_SK6812_EC15_1.5x1.5mm, F.Cu at (103.1, 72.6)
- added D9: SK6805-EC15, LED_SMD:LED_SK6812_EC15_1.5x1.5mm, F.Cu at (123.1, 70.1)
- added H1: MountingHole, MountingHole:MountingHole_2.2mm_M2_ISO7380, F.Cu at (80.9, 132.4)
- added H2: MountingHole, MountingHole:MountingHole_2.2mm_M2_ISO7380, F.Cu at (174.8, 90.4)
- added J1: Conn_01x04_Pin, Connector_JST:JST_PH_B4B-PH-K_1x04_P2.00mm_Vertical, F.Cu at (197.0, 124.8)
- added J3: XT60PW-M, Connector_AMASS:AMASS_XT60PW-M_1x02_P7.20mm_Horizontal, F.Cu at (190.9, 95.9)
- added L3: 4n7, Inductor_SMD:L_0402_1005Metric_Pad0.77x0.64mm_HandSolder, F.Cu at (186.5, 104.8)
- added L4: 2n2, Inductor_SMD:L_0402_1005Metric_Pad0.77x0.64mm_HandSolder, F.Cu at (187.2, 106.5)
- added Q1: NTJD4152PT1G, Package_TO_SOT_SMD:SOT-363_SC-70-6_Handsoldering, F.Cu at (174.5, 125.5)
- added Q2: NTJD4152PT1G, Package_TO_SOT_SMD:SOT-363_SC-70-6_Handsoldering, F.Cu at (220.5, 114.0)
- added Q3: Q_Dual_NMOS_S1G1D2S2G2D1, Package_TO_SOT_SMD:SOT-363_SC-70-6, F.Cu at (189.0, 124.5)
- added Q8: NTJD4152PT1G, Package_TO_SOT_SMD:SOT-363_SC-70-6_Handsoldering, F.Cu at (177.5, 125.5)
- added R1: 100R, Resistor_SMD:R_0402_1005Metric_Pad0.72x0.64mm_HandSolder, F.Cu at (179.8, 110.5)
- added R16: 330R, Resistor_SMD:R_0402_1005Metric_Pad0.72x0.64mm_HandSolder, F.Cu at (193.1, 119.5)
- added R18: 20k, Resistor_SMD:R_0402_1005Metric_Pad0.72x0.64mm_HandSolder, F.Cu at (193.1, 121.5)
- added R2: 50k, Resistor_SMD:R_0402_1005Metric_Pad0.72x0.64mm_HandSolder, F.Cu at (179.2, 134.0)
- added R25: 100R, Resistor_SMD:R_0402_1005Metric_Pad0.72x0.64mm_HandSolder, F.Cu at (178.8, 110.5)
- added R26: 4k7, Resistor_SMD:R_0402_1005Metric_Pad0.72x0.64mm_HandSolder, F.Cu at (177.8, 110.5)
- added R28: 0R, Resistor_SMD:R_0402_1005Metric_Pad0.72x0.64mm_HandSolder, F.Cu at (176.0, 99.5)
- added R29: 0R, Resistor_SMD:R_0402_1005Metric_Pad0.72x0.64mm_HandSolder, F.Cu at (177.0, 99.5)
- added SW1: MK-12C02-G020, Button_Switch_SMD:SW_SPDT_PCM12, F.Cu at (177.3, 137.5)
- added TP3: TestPoint, TestPoint:TestPoint_Pad_D1.0mm, F.Cu at (196.5, 112.2)
- added U2: TMUX1208RSV, Package_DFN_QFN:UQFN-16_1.8x2.6mm_P0.4mm, F.Cu at (213.9, 112.2)
- added U6: MCP73831-2-OT, Package_TO_SOT_SMD:SOT-23-5, F.Cu at (188.9, 121.0)
- added U8: nRF52833_QDxx, Package_DFN_QFN:QFN-40-1EP_5x5mm_P0.4mm_EP3.6x3.6mm, F.Cu at (179.4, 104.2)
- added Y1: 32MHz, Crystal:Crystal_SMD_2016-4Pin_2.0x1.6mm, F.Cu at (186.4, 101.7)
- added Y2: 32768 KHz, Crystal:Crystal_SMD_2012-2Pin_2.0x1.2mm_HandSoldering, F.Cu at (173.5, 103.7)
- C10: renamed from C109; footprint Capacitor_SMD:C_0603_1608Metric_Pad1.08x0.95mm_HandSolder -> Capacitor_SMD:C_0402_1005Metric_Pad0.74x0.62mm_HandSolder
- C11: renamed from C110; footprint Capacitor_SMD:C_0603_1608Metric_Pad1.08x0.95mm_HandSolder -> Capacitor_SMD:C_0402_1005Metric_Pad0.74x0.62mm_HandSolder
- C13: renamed from C112; footprint Capacitor_SMD:CP_Elec_6.3x7.7 -> Capacitor_Tantalum_SMD:CP_EIA-6032-28_Kemet-C_HandSolder
- C14: renamed from C113; footprint Capacitor_SMD:C_0603_1608Metric_Pad1.08x0.95mm_HandSolder -> Capacitor_SMD:C_0402_1005Metric_Pad0.74x0.62mm_HandSolder
- C15: renamed from C114; footprint Capacitor_SMD:C_0603_1608Metric_Pad1.08x0.95mm_HandSolder -> Capacitor_SMD:C_0402_1005Metric_Pad0.74x0.62mm_HandSolder
- C16: renamed from C201; footprint Capacitor_SMD:C_0603_1608Metric_Pad1.08x0.95mm_HandSolder -> Capacitor_SMD:C_0402_1005Metric_Pad0.74x0.62mm_HandSolder
- C17: renamed from C202; footprint Capacitor_SMD:C_0603_1608Metric_Pad1.08x0.95mm_HandSolder -> Capacitor_SMD:C_0402_1005Metric_Pad0.74x0.62mm_HandSolder
- C18: renamed from C203; footprint Capacitor_SMD:C_0603_1608Metric_Pad1.08x0.95mm_HandSolder -> Capacitor_SMD:C_0402_1005Metric_Pad0.74x0.62mm_HandSolder
- C19: renamed from C204; footprint Capacitor_SMD:C_0603_1608Metric_Pad1.08x0.95mm_HandSolder -> Capacitor_SMD:C_0402_1005Metric_Pad0.74x0.62mm_HandSolder
- C20: renamed from C205; footprint Capacitor_SMD:C_0603_1608Metric_Pad1.08x0.95mm_HandSolder -> Capacitor_SMD:C_0402_1005Metric_Pad0.74x0.62mm_HandSolder
- C21: renamed from C206; footprint Capacitor_SMD:C_0603_1608Metric_Pad1.08x0.95mm_HandSolder -> Capacitor_SMD:C_0402_1005Metric_Pad0.74x0.62mm_HandSolder
- C22: renamed from C207; footprint Capacitor_SMD:C_0603_1608Metric_Pad1.08x0.95mm_HandSolder -> Capacitor_SMD:C_0402_1005Metric_Pad0.74x0.62mm_HandSolder
- C23: renamed from C208; footprint Capacitor_SMD:C_0603_1608Metric_Pad1.08x0.95mm_HandSolder -> Capacitor_SMD:C_0402_1005Metric_Pad0.74x0.62mm_HandSolder
- C24: renamed from C209; footprint Capacitor_SMD:C_0603_1608Metric_Pad1.08x0.95mm_HandSolder -> Capacitor_SMD:C_0402_1005Metric_Pad0.74x0.62mm_HandSolder
- C25: renamed from C210; footprint Capacitor_SMD:C_0603_1608Metric_Pad1.08x0.95mm_HandSolder -> Capacitor_SMD:C_0402_1005Metric_Pad0.74x0.62mm_HandSolder
- C26: renamed from C211; footprint Capacitor_SMD:C_0603_1608Metric_Pad1.08x0.95mm_HandSolder -> Capacitor_SMD:C_0402_1005Metric_Pad0.74x0.62mm_HandSolder
- C27: renamed from C212; footprint Capacitor_SMD:C_0603_1608Metric_Pad1.08x0.95mm_HandSolder -> Capacitor_SMD:C_0402_1005Metric_Pad0.74x0.62mm_HandSolder
- C28: renamed from C213; footprint Capacitor_SMD:C_0603_1608Metric_Pad1.08x0.95mm_HandSolder -> Capacitor_SMD:C_0402_1005Metric_Pad0.74x0.62mm_HandSolder
- C29: renamed from C214; footprint Capacitor_SMD:C_0603_1608Metric_Pad1.08x0.95mm_HandSolder -> Capacitor_SMD:C_0402_1005Metric_Pad0.74x0.62mm_HandSolder
- C30: renamed from C215; footprint Capacitor_SMD:C_0603_1608Metric_Pad1.08x0.95mm_HandSolder -> Capacitor_SMD:C_0402_1005Metric_Pad0.74x0.62mm_HandSolder
- C31: renamed from C216; footprint Capacitor_SMD:C_0603_1608Metric_Pad1.08x0.95mm_HandSolder -> Capacitor_SMD:C_0402_1005Metric_Pad0.74x0.62mm_HandSolder
- C32: renamed from C217; footprint Capacitor_SMD:C_0603_1608Metric_Pad1.08x0.95mm_HandSolder -> Capacitor_SMD:C_0402_1005Metric_Pad0.74x0.62mm_HandSolder
- C33: renamed from C218; footprint Capacitor_SMD:C_0603_1608Metric_Pad1.08x0.95mm_HandSolder -> Capacitor_SMD:C_0402_1005Metric_Pad0.74x0.62mm_HandSolder
- C34: renamed from C219; footprint Capacitor_SMD:C_0603_1608Metric_Pad1.08x0.95mm_HandSolder -> Capacitor_SMD:C_0402_1005Metric_Pad0.74x0.62mm_HandSolder
- C7: renamed from C107; footprint Capacitor_SMD:C_0603_1608Metric_Pad1.08x0.95mm_HandSolder -> Capacitor_SMD:C_0402_1005Metric_Pad0.74x0.62mm_HandSolder
- C8: renamed from C108; footprint Capacitor_SMD:C_0603_1608Metric_Pad1.08x0.95mm_HandSolder -> Capacitor_SMD:C_0402_1005Metric_Pad0.74x0.62mm_HandSolder
- R10: renamed from R108; value 330R -> 50k; footprint Resistor_SMD:R_0603_1608Metric_Pad0.98x0.95mm_HandSolder -> Resistor_SMD:R_0402_1005Metric_Pad0.72x0.64mm_HandSolder
- R12: renamed from R110; value 2k2 -> 50k; footprint Resistor_SMD:R_0603_1608Metric_Pad0.98x0.95mm_HandSolder -> Resistor_SMD:R_0402_1005Metric_Pad0.72x0.64mm_HandSolder
- R13: renamed from R111; value 50k -> 33k; footprint Resistor_SMD:R_0603_1608Metric_Pad0.98x0.95mm_HandSolder -> Resistor_SMD:R_0402_1005Metric_Pad0.72x0.64mm_HandSolder
- R14: renamed from R112; value 33k -> 51k; footprint Resistor_SMD:R_0603_1608Metric_Pad0.98x0.95mm_HandSolder -> Resistor_SMD:R_0402_1005Metric_Pad0.72x0.64mm_HandSolder
- R15: renamed from R113; value 51k -> 56k; footprint Resistor_SMD:R_0603_1608Metric_Pad0.98x0.95mm_HandSolder -> Resistor_SMD:R_0402_1005Metric_Pad0.72x0.64mm_HandSolder
- R17: renamed from R114; value 56k -> 330R; footprint Resistor_SMD:R_0603_1608Metric_Pad0.98x0.95mm_HandSolder -> Resistor_SMD:R_0402_1005Metric_Pad0.72x0.64mm_HandSolder
- R21: renamed from R201; footprint Resistor_SMD:R_0603_1608Metric_Pad0.98x0.95mm_HandSolder -> Resistor_SMD:R_0402_1005Metric_Pad0.72x0.64mm_HandSolder
- R22: renamed from R202; footprint Resistor_SMD:R_0603_1608Metric_Pad0.98x0.95mm_HandSolder -> Resistor_SMD:R_0402_1005Metric_Pad0.72x0.64mm_HandSolder
- R23: renamed from R203; footprint Resistor_SMD:R_0603_1608Metric_Pad0.98x0.95mm_HandSolder -> Resistor_SMD:R_0402_1005Metric_Pad0.72x0.64mm_HandSolder
- R24: renamed from R204; footprint Resistor_SMD:R_0603_1608Metric_Pad0.98x0.95mm_HandSolder -> Resistor_SMD:R_0402_1005Metric_Pad0.72x0.64mm_HandSolder
- R3: renamed from R101; value 50k -> 5k1; footprint Resistor_SMD:R_0603_1608Metric_Pad0.98x0.95mm_HandSolder -> Resistor_SMD:R_0402_1005Metric_Pad0.72x0.64mm_HandSolder
- R4: renamed from R102; footprint Resistor_SMD:R_0603_1608Metric_Pad0.98x0.95mm_HandSolder -> Resistor_SMD:R_0402_1005Metric_Pad0.72x0.64mm_HandSolder
- R5: renamed from R103; value 5k1 -> 0R; footprint Resistor_SMD:R_0603_1608Metric_Pad0.98x0.95mm_HandSolder -> Resistor_SMD:R_0402_1005Metric_Pad0.72x0.64mm_HandSolder
- R6: renamed from R104; value 0R -> 110k; footprint Resistor_SMD:R_0603_1608Metric_Pad0.98x0.95mm_HandSolder -> Resistor_SMD:R_0402_1005Metric_Pad0.72x0.64mm_HandSolder
- R7: renamed from R105; value 110k -> 15k; footprint Resistor_SMD:R_0603_1608Metric_Pad0.98x0.95mm_HandSolder -> Resistor_SMD:R_0402_1005Metric_Pad0.72x0.64mm_HandSolder
- U7: renamed from U107; footprint Package_SO:SOIC-8_3.9x4.9mm_P1.27mm -> Package_DFN_QFN:DFN-8-1EP_2x2mm_P0.5mm_EP1.05x1.75mm
- moved SW19 285.6 mm to (143.1, 127.1)
- moved SW20 285.6 mm to (163.1, 129.6)
- moved C34 285.6 mm to (159.2, 138.2)
- moved D44 285.6 mm to (163.1, 138.4)
- moved C33 285.5 mm to (139.2, 135.7)
- moved D43 285.5 mm to (143.1, 135.9)
- moved C31 285.4 mm to (99.2, 135.7)
- moved D41 285.4 mm to (103.1, 135.9)
- moved SW17 285.4 mm to (103.1, 127.1)
- moved SW18 285.4 mm to (123.1, 124.6)
- moved C32 285.3 mm to (119.2, 133.2)
- moved D42 285.3 mm to (123.1, 133.4)
- moved C16 265.5 mm to (79.2, 78.2)
- moved C17 265.5 mm to (99.2, 75.7)
- moved C18 265.5 mm to (119.2, 73.2)
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- renumbered BT101 to BT1, D101 to D1, D201 to D12, D202 to D13, D203 to D14, D204 to D15, D205 to D16, D102 to D2, D206 to D22, D207 to D23, D208 to D24, D209 to D25, D210 to D26, D211 to D32, D212 to D33, D213 to D34, D214 to D35, D215 to D36, D216 to D41, D217 to D42, D218 to D43, D219 to D44, D105 to D5, D106 to D6, F101 to F1, L102 to L1, L103 to L2, SW209 to SW10, SW210 to SW11, SW211 to SW12, SW212 to SW13, SW213 to SW14, SW214 to SW15, SW215 to SW16, SW216 to SW17, SW217 to SW18, SW218 to SW19, SW201 to SW2, SW219 to SW20, SW202 to SW3, SW203 to SW4, SW204 to SW5, SW205 to SW6, SW206 to SW7, SW207 to SW8, SW208 to SW9, TP101 to TP1, TP103 to TP2, U101 to U1, U103 to U3, U104 to U4, USB101 to USB1
Connections:
- C14 pad 1: +5V -> +3V3
- D5 pad 1: Net-(D105-K) -> Net-(D5-K)
- D6 pad 2: Net-(D106-A) -> Net-(D6-A)
- R10 pad 1: +3V3USB -> Net-(Q2A-G)
- R10 pad 2: Net-(D104-A) -> /VBAT
- R12 pad 1: Net-(U105-PROG) -> /VBAT
- R12 pad 2: GND -> +3V3USB
- R13 pad 2: +3V3USB -> Net-(U7A-+)
- R14 pad 2: Net-(U107A-+) -> Net-(D5-K)
- R15 pad 1: /VBAT -> Net-(U7A-+)
- R15 pad 2: Net-(D105-K) -> GND
- R17 pad 1: Net-(U107A-+) -> Net-(R17-Pad1)
- R17 pad 2: GND -> Net-(D6-A)
- R21 pad 1: /Matrix/LEDDATA0 -> /LD0
- R22 pad 1: /Matrix/LEDDATA1 -> /LD1
- R23 pad 1: /Matrix/LEDDATA2 -> /LD2
- R24 pad 1: /Matrix/LEDDATA3 -> /LD3
- R3 pad 1: /LEDTOGGLE -> Net-(USB1-CC2)
- R4 pad 1: Net-(USB101-CC2) -> Net-(USB1-CC1)
- R5 pad 1: Net-(USB101-CC1) -> +5VUSB
- R5 pad 2: GND -> Net-(U3-EN)
- R6 pad 1: +5VUSB -> +5VBAT
- R6 pad 2: Net-(U103-EN) -> Net-(U4-FB)
- R7 pad 1: +5VBAT -> Net-(U4-FB)
- R7 pad 2: Net-(U104-FB) -> GND
- SW10 pad 1: /COL1 -> /COL3
- SW11 pad 1: /COL0 -> /COL4
- SW12 pad 1: /COL4 -> /COL0
- SW13 pad 1: /COL3 -> /COL1
- SW15 pad 1: /COL1 -> /COL3
- SW16 pad 1: /COL0 -> /COL4
- SW17 pad 1: /COL4 -> /COL1
- SW18 pad 1: unconnected-(SW217-Pad1) -> /COL2
- SW19 pad 1: unconnected-(SW218-Pad1) -> /COL3
- SW2 pad 1: /COL4 -> /COL0
- SW20 pad 1: unconnected-(SW219-Pad1) -> /COL4
- SW3 pad 1: /COL3 -> /COL1
- SW5 pad 1: /COL1 -> /COL3
- SW6 pad 1: /COL0 -> /COL4
- SW7 pad 1: /COL4 -> /COL0
- SW8 pad 1: /COL3 -> /COL1
- TP2 pad 1: +3V3USB -> +5VUSB
- U3 pad 3: Net-(U103-EN) -> Net-(U3-EN)
- U4 pad 3: Net-(U104-FB) -> Net-(U4-FB)
- U7 pad 1: Net-(R115-Pad1) -> Net-(R17-Pad1)
- U7 pad 2: Net-(D105-K) -> Net-(D5-K)
- U7 pad 3: Net-(U107A-+) -> Net-(U7A-+)
- USB1 pad 10: Net-(USB101-CC2) -> Net-(USB1-CC2)
- USB1 pad 4: Net-(USB101-CC1) -> Net-(USB1-CC1)
Routing:
- net /D-: track 0.00 -> 48.6 mm, vias 0 -> 4
- net /D+: track 0.00 -> 48.2 mm, vias 0 -> 4
- net Net-(U8-XC2): track 0.00 -> 6.76 mm
- net Net-(U8-ANT): track 0.00 -> 5.81 mm
- net Net-(U8-XC1): track 0.00 -> 4.20 mm
- net Net-(U8-XL2/P0.01): track 0.00 -> 4.10 mm
- net /LEDSEL1: track 0.00 -> 3.77 mm
- net Net-(U8-XL1/P0.00): track 0.00 -> 3.70 mm
- net /LEDSEL0: track 0.00 -> 3.19 mm
- net Net-(U8-DEC5): track 0.00 -> 2.47 mm
- net Net-(C40-Pad1): track 0.00 -> 2.25 mm
- net Net-(AE1-A): track 0.00 -> 2.21 mm
- net Net-(U8-DEC4): track 0.00 -> 0.96 mm
- removed copper zone on B.Cu, net GND
Other:
- board size 663.8 x 129.9 mm -> 125 x 85 mm
- board text added: "0"
- board text added: "0 mm"
- board text added: "0.01 mm"
- board text added: "0.02"
- board text added: "0.035 mm"
- board text added: "1"
- board text added: "1.51 mm"
- board text added: "3.3"
- board text added: "4.5"
- board text added: "B.Cu"
- board text added: "B.Mask"
- board text added: "B.Paste"
- board text added: "B.Silkscreen"
- board text added: "Bottom Silk Screen"
- board text added: "Bottom Solder Mask"
- board text added: "Bottom Solder Paste"
- board text added: "Color"
- board text added: "Dielectric 1"
- board text added: "Epsilon R"
- board text added: "F.Cu"
- board text added: "F.Mask"
- board text added: "F.Paste"
- board text added: "F.Silkscreen"
- board text added: "FR4"
- board text added: "Layer Name"
- board text added: "Loss Tangent"
- board text added: "Material"
- board text added: "Not specified"
- board text added: "Thickness (mm)"
- board text added: "Top Silk Screen"
- board text added: "Top Solder Mask"
- board text added: "Top Solder Paste"
- board text added: "Type"
- board text added: "copper"
- board text added: "core"
